Commit message: port, not working

File: mir_description/urdf/include/caster.urdf.xacro (robot description, xacro)
@@ -12,9 +12,6 @@
     </joint>
     <gazebo>
-      <plugin name="${locationprefix}_caster_rotation_joint_states" filename="libgazebo_ros_joint_state_publisher.so">
-        <ros>
-          <namespace>${ns}</namespace>
-        </ros>
-        <update_rate>200.0</update_rate>
+      <plugin filename="gz-sim-joint-state-publisher-system" name="gz::sim::systems::JointStatePublisher">
+        <namespace>${ns}</namespace>
         <joint_name>${prefix}${locationprefix}_caster_rotation_joint</joint_name>
       </plugin>
@@ -58,9 +55,6 @@
     </joint>
     <gazebo>
-      <plugin name="${locationprefix}_caster_wheel_joint_states" filename="libgazebo_ros_joint_state_publisher.so">
-        <ros>
-          <namespace>${ns}</namespace>
-        </ros>
-        <update_rate>200.0</update_rate>
+      <plugin filename="gz-sim-joint-state-publisher-system" name="gz::sim::systems::JointStatePublisher">
+        <namespace>${ns}</namespace>
         <joint_name>${prefix}${locationprefix}_caster_wheel_joint</joint_name>
       </plugin>

File: mir_description/urdf/include/common.gazebo.xacro (robot description, xacro)
@@ -3,5 +3,5 @@
   <xacro:macro name="controller_plugin_gazebo" params="robot_namespace">
     <gazebo>
-      <plugin filename="libgazebo_ros2_control.so" name="gazebo_ros2_control">
+      <plugin filename="gz_ros2_control-system" name="gz_ros2_control::GazeboSimROS2ControlPlugin">
         <robot_param>robot_description</robot_param>
         <robot_param_node>robot_state_publisher</robot_param_node>

File: mir_description/urdf/include/imu.gazebo.urdf.xacro (robot description, xacro)
@@ -17,4 +17,6 @@
         <update_rate>${update_rate}</update_rate>
         <visualize>true</visualize>
+        <frame_id>${imu_frame}</frame_id>
+        <topic>${imu_topic}</topic>
         <imu>
           <angular_velocity>
@@ -71,12 +73,4 @@
           </linear_acceleration>
         </imu>
-        <plugin filename="libgazebo_ros_imu_sensor.so" name="imu_plugin">
-        <initial_orientation_as_reference>false</initial_orientation_as_reference>
-          <ros>
-            <namespace>${imu_topic}</namespace>
-            <remapping>~/out:=data</remapping>
-            <frame_name>${imu_frame}</frame_name>  <!-- from real MiR -->
-          </ros>
-        </plugin>
       </sensor>
     </gazebo>

File: mir_description/urdf/include/mir_100.gazebo.xacro (robot description, xacro)
@@ -26,5 +26,5 @@
   </xacro:macro>
  <!-- See https://github.com/ros-simulation/gazebo_ros_pkgs/wiki/ROS-2-Migration:-P3D for ros2 information -->
-  <xacro:macro name="p3d_base_controller" params="prefix">
+  <!-- <xacro:macro name="p3d_base_controller" params="prefix">
     <gazebo>
       <plugin name="p3d_base_controller" filename="libgazebo_ros_p3d.so">
@@ -41,4 +41,4 @@
       </plugin>
     </gazebo>
-  </xacro:macro>
+  </xacro:macro> -->
 </robot>

File: mir_description/urdf/include/sick_s300.urdf.xacro (robot description, xacro)
@@ -29,8 +29,10 @@
       <!-- <material value="Gazebo/Yellow" /> -->
       <material value="Gazebo/FlatBlack" />
-      <sensor type="ray" name="${prefix}${link}">
+      <sensor type="gpu_lidar" name="${prefix}${link}">
         <visualize>false</visualize>
         <update_rate>12.5</update_rate>
-        <ray>
+        <frame_id>${prefix}${link}</frame_id>
+        <topic>${prefix}${topic}</topic>
+        <lidar>
           <scan>
             <horizontal>
@@ -54,6 +56,6 @@
             <stddev>0.01</stddev>
           </noise>
-        </ray>
-        <plugin name="gazebo_ros_${link}_controller" filename="libgazebo_ros_ray_sensor.so">
+        </lidar>
+        <!-- <plugin name="gazebo_ros_${link}_controller" type="libgazebo_ros_ray_sensor.so">
           <ros>
             <remapping>~/out:=${prefix}${topic}</remapping>
@@ -61,5 +63,5 @@
           <output_type>sensor_msgs/LaserScan</output_type>
           <frame_name>${prefix}${link}</frame_name>
-        </plugin>
+        </plugin> -->
       </sensor>
     </gazebo>

Commit message: rviz looks fine, tf lookup error

File: mir_description/urdf/include/caster.urdf.xacro (robot description, xacro)
@@ -14,4 +14,5 @@
       <plugin filename="gz-sim-joint-state-publisher-system" name="gz::sim::systems::JointStatePublisher">
         <namespace>${ns}</namespace>
+        <topic>joint_states</topic>
         <joint_name>${prefix}${locationprefix}_caster_rotation_joint</joint_name>
       </plugin>
@@ -57,4 +58,5 @@
       <plugin filename="gz-sim-joint-state-publisher-system" name="gz::sim::systems::JointStatePublisher">
         <namespace>${ns}</namespace>
+        <topic>joint_states</topic>
         <joint_name>${prefix}${locationprefix}_caster_wheel_joint</joint_name>
       </plugin>

File: mir_description/urdf/include/mir_100.gazebo.xacro (robot description, xacro)
@@ -25,20 +25,3 @@
     </gazebo>
   </xacro:macro>
- <!-- See https://github.com/ros-simulation/gazebo_ros_pkgs/wiki/ROS-2-Migration:-P3D for ros2 information -->
-  <!-- <xacro:macro name="p3d_base_controller" params="prefix">
-    <gazebo>
-      <plugin name="p3d_base_controller" filename="libgazebo_ros_p3d.so">
-        <ros>
-          <remapping>odom:=${prefix}base_pose_ground_truth</remapping>
-        </ros>
-        <always_on>true</always_on>
-        <update_rate>50.0</update_rate>
-        <body_name>${prefix}base_footprint</body_name>
-        <gaussian_noise>0.01</gaussian_noise>
-        <frame_name>map</frame_name>
-        <xyz_offset>0 0 0</xyz_offset>
-        <rpy_offset>0 0 0</rpy_offset>
-      </plugin>
-    </gazebo>
-  </xacro:macro> -->
 </robot>

File: mir_description/urdf/include/mir_100_v1.urdf.xacro (robot description, xacro)
@@ -141,5 +141,4 @@
     <link name="${prefix}surface_mount"/>
     <xacro:mir_100_wheel_transmissions prefix="${prefix}"/>
-    <xacro:p3d_base_controller prefix="${prefix}"/>
   </xacro:macro>
 </robot>
